Commit message: commit

File: urdf/my_robot.xacro (robot description, xacro)
@@ -148,5 +148,5 @@
   <parent link="base_link"/>
   <child link="wheel_rf_1"/>
-  <axis xyz="0.0 1.0 0.0"/>
+  <axis xyz="0.0 -1.0 0.0"/>
 </joint>
 <joint name="motor_rb" type="continuous">
@@ -154,5 +154,5 @@
   <parent link="base_link"/>
   <child link="wheel_rb_1"/>
-  <axis xyz="0.0 1.0 0.0"/>
+  <axis xyz="0.0 -1.0 0.0"/>
 </joint>
 <joint name="motor_lb" type="continuous">
